Commit message: Exercise 3.10
Last touch on the last assignment.\nAdding another lower arm and an elbow joint with a motor.

File: catkin_ws/src/hello_ros/urdf/hello_gazebo_robot_2.urdf (robot description, URDF)
Before this commit: robot hello_ros_robot, 4 links, 3 joints
Links:
- added link lower_arm, mass 1.0; collision cylinder length=0.4 radius=0.05; visual cylinder length=0.4 radius=0.05
Joints:
- added joint elbow: type continuous, parent upper_arm, child lower_arm, origin xyz=0.0 -0.1 0.45 rpy=0 1.5708 0, axis 0 1 0
